Commit message: Initial commit

File: src/robot_description/src/description/robot_description.urdf (robot description, URDF)
Before this commit: robot robot, 3 links, 2 joints
Links:
- added link laser_frame; visual sphere radius=${(wheel_radius+wheel_zoff-(base_height/2))}
Joints:
- added joint laser_link: type fixed, parent base_link, child laser_frame, origin xyz=0.0 0.0 ${(base_height-(wheel_radius+wheel_zoff-(base_height/2)))} rpy=0 0 0
