Commit message: Rebuild on Humble and publish the real robomo frames
The image was FROM frankjoshua/ros2 - a floating tag that got rebuilt on
Jazzy, whose Fast DDS wire format corrupts discovery for the Humble robot
stack (slam drops every scan -> no map, nav2 throws extrapolation errors).
Pin FROM ros:humble-ros-base directly so the distro can't drift.

Replace the generic tutorial box-robot URDF (laser at ~0.18 m, no camera/
imu/gps) with the real robomo frames - laser_frame at 0.03,0,1.23 plus
camera/imu/gps - as self-contained primitives (no mesh server needed).
Simplify to robot_state_publisher only: the URDF is plain, all-fixed-joint,
so no xacro / joint_state_publisher, and launch without the interactive
bashrc.

Co-Authored-By: Claude Opus 4.8 (1M context) <noreply@anthropic.com>

File: ros2_ws/src/robot_description/src/description/robot_description.urdf (robot description, URDF)
Before this commit: robot robot, 4 links, 3 joints
Links:
- removed link front_caster
- added link camera_link; visual box size=0.025 0.09 0.025
- added link camera_optical_frame
- added link drivewhl_l_link; visual cylinder length=0.04 radius=0.10
- added link drivewhl_r_link; visual cylinder length=0.04 radius=0.10
- added link gps_link
- added link imu_link
- link base_link: geometry visual box size=0.42 0.31 0.20; visual cylinder length=1.02 radius=0.03
- link laser_frame: geometry visual cylinder length=0.04 radius=0.04
Joints:
- removed joint base_joint
- removed joint caster_joint
- removed joint laser_link
- added joint base_footprint_joint: type fixed, parent base_link, child base_footprint, origin xyz=0 0 0 rpy=0 0 0
- added joint camera_joint: type fixed, parent base_link, child camera_link, origin xyz=0.31 0 0.28 rpy=0 0 0
- added joint camera_optical_joint: type fixed, parent camera_link, child camera_optical_frame, origin xyz=0 0 0 rpy=-1.5708 0 -1.5708
- added joint drivewhl_l_joint: type fixed, parent base_link, child drivewhl_l_link, origin xyz=-0.12 0.18 0.10 rpy=0 0 0
- added joint drivewhl_r_joint: type fixed, parent base_link, child drivewhl_r_link, origin xyz=-0.12 -0.18 0.10 rpy=0 0 0
- added joint gps_joint: type fixed, parent base_link, child gps_link, origin xyz=0.07 -0.02 0.60 rpy=0 0 0
- added joint imu_joint: type fixed, parent base_link, child imu_link, origin xyz=0.05 0.08 0.594 rpy=0 0 0
- added joint laser_joint: type fixed, parent base_link, child laser_frame, origin xyz=0.03 0 1.23 rpy=0 0 0
